File: PCB/key_column.kicad_pcb (KiCad board)
At the start: 2 copper layers, 6 parts, among them SW1201 SW_Push, U1201 SK6812MINI-E_C5149201

Commit message: Removed 8-key units, now using the PCB view to handle routing the keys to the SOIP shift registers.
Changed lines of the file:
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@@
   (segment (start 28.2 21) (end 28.200102 22.119898) (width 0.5) (layer "B.Cu") (net 2))
   (segment (start 30.8 21.6) (end 30.8 21.12) (width 0.5) (layer "B.Cu") (net 3))
-  (segment (start 31.2 21.6) (end 32.4 22.8) (width 0.5) (layer "B.Cu") (net 3))
+  (segment (start 31.2 21.6) (end 32.4 22.8) (width 0.2) (layer "B.Cu") (net 3))
   (segment (start 30.8 21.6) (end 31.2 21.6) (width 0.5) (layer "B.Cu") (net 3))
   (segment (start 30.8 21.12) (end 30.92 21) (width 0.5) (layer "B.Cu") (net 3))
