File: PCB/PCB.kicad_pcb (KiCad board)
At the start: 2 copper layers, 182.9 x 104.1 mm, 33 parts, among them SW1 SW_Push, SW2 SW_Push, SW3 SW_Push, SW4 SW_Push, SW5 SW_Push, SW6 SW_Push, SW7 SW_Push, SW8 SW_Push

Commit message: Ready to work on PCB
Parts:
- added C10: 4.7uF, Capacitor_SMD:C_0603_1608Metric, F.Cu at (63.1, 63.8)
- added C11: 100nF, Capacitor_SMD:C_0402_1005Metric, F.Cu at (69.4, 44.5)
- added C12: 100nF, Capacitor_SMD:C_0402_1005Metric, F.Cu at (69.4, 46.4)
- added C13: 100uF, Capacitor_Tantalum_SMD:CP_EIA-3528-15_AVX-H, F.Cu at (73.9, 60.9)
- added C14: 100uF, Capacitor_Tantalum_SMD:CP_EIA-3528-15_AVX-H, F.Cu at (73.9, 65.3)
- added C9: 1uF, Capacitor_SMD:C_0402_1005Metric, F.Cu at (69.4, 42.5)
- added CL1: 100nF, Capacitor_SMD:C_0402_1005Metric, F.Cu at (126.0, 107.8)
- added CL10: 100nF, Capacitor_SMD:C_0402_1005Metric, F.Cu at (202.8, 86.0)
- added CL11: 100nF, Capacitor_SMD:C_0402_1005Metric, F.Cu at (145.2, 151.5)
- added CL12: 100nF, Capacitor_SMD:C_0402_1005Metric, F.Cu at (106.8, 86.0)
- added CL13: 100nF, Capacitor_SMD:C_0402_1005Metric, F.Cu at (123.5, 54.1)
- added CL14: 100nF, Capacitor_SMD:C_0402_1005Metric, F.Cu at (145.2, 86.0)
- added CL15: 100nF, Capacitor_SMD:C_0402_1005Metric, F.Cu at (87.6, 129.7)
- added CL16: 100nF, Capacitor_SMD:C_0402_1005Metric, F.Cu at (68.4, 107.8)
- added CL17: 100nF, Capacitor_SMD:C_0402_1005Metric, F.Cu at (87.6, 151.5)
- added CL18: 100nF, Capacitor_SMD:C_0402_1005Metric, F.Cu at (106.8, 173.3)
- added CL19: 100nF, Capacitor_SMD:C_0402_1005Metric, F.Cu at (181.1, 54.1)
- added CL2: 100nF, Capacitor_SMD:C_0402_1005Metric, F.Cu at (68.4, 151.5)
- added CL20: 100nF, Capacitor_SMD:C_0402_1005Metric, F.Cu at (145.2, 173.3)
- added CL21: 100nF, Capacitor_SMD:C_0402_1005Metric, F.Cu at (106.8, 107.8)
- added CL22: 100nF, Capacitor_SMD:C_0402_1005Metric, F.Cu at (183.6, 151.5)
- added CL23: 100nF, Capacitor_SMD:C_0402_1005Metric, F.Cu at (164.4, 86.0)
- added CL24: 100nF, Capacitor_SMD:C_0402_1005Metric, F.Cu at (142.7, 54.1)
- added CL25: 100nF, Capacitor_SMD:C_0402_1005Metric, F.Cu at (87.6, 107.8)
- added CL26: 100nF, Capacitor_SMD:C_0402_1005Metric, F.Cu at (202.8, 107.8)
- added CL27: 100nF, Capacitor_SMD:C_0402_1005Metric, F.Cu at (126.0, 129.7)
- added CL28: 100nF, Capacitor_SMD:C_0402_1005Metric, F.Cu at (126.0, 86.0)
- added CL29: 100nF, Capacitor_SMD:C_0402_1005Metric, F.Cu at (145.2, 107.8)
- added CL3: 100nF, Capacitor_SMD:C_0402_1005Metric, F.Cu at (202.8, 151.5)
- added CL30: 100nF, Capacitor_SMD:C_0402_1005Metric, F.Cu at (161.9, 54.1)
- added CL31: 100nF, Capacitor_SMD:C_0402_1005Metric, F.Cu at (87.6, 173.3)
- added CL32: 100nF, Capacitor_SMD:C_0402_1005Metric, F.Cu at (145.2, 129.7)
- added CL33: 100nF, Capacitor_SMD:C_0402_1005Metric, F.Cu at (68.4, 173.3)
- added CL34: 100nF, Capacitor_SMD:C_0402_1005Metric, F.Cu at (126.0, 151.5)
- added CL35: 100nF, Capacitor_SMD:C_0402_1005Metric, F.Cu at (164.4, 151.5)
- added CL36: 100nF, Capacitor_SMD:C_0402_1005Metric, F.Cu at (183.6, 129.7)
- added CL37: 100nF, Capacitor_SMD:C_0402_1005Metric, F.Cu at (164.4, 129.7)
- added CL38: 100nF, Capacitor_SMD:C_0402_1005Metric, F.Cu at (87.6, 86.0)
- added CL39: 100nF, Capacitor_SMD:C_0402_1005Metric, F.Cu at (106.8, 151.5)
- added CL4: 100nF, Capacitor_SMD:C_0402_1005Metric, F.Cu at (183.6, 107.8)
- added CL40: 100nF, Capacitor_SMD:C_0402_1005Metric, F.Cu at (126.0, 173.3)
- added CL41: 100nF, Capacitor_SMD:C_0402_1005Metric, F.Cu at (68.4, 129.7)
- added CL43: 100nF, Capacitor_SMD:C_0402_1005Metric, F.Cu at (200.3, 54.1)
- added CL45: 100nF, Capacitor_SMD:C_0402_1005Metric, F.Cu at (164.4, 173.3)
- added CL46: 100nF, Capacitor_SMD:C_0402_1005Metric, F.Cu at (202.8, 173.3)
- added CL47: 100nF, Capacitor_SMD:C_0402_1005Metric, F.Cu at (106.8, 129.7)
- added CL5: 100nF, Capacitor_SMD:C_0402_1005Metric, F.Cu at (164.4, 107.8)
- added CL6: 100nF, Capacitor_SMD:C_0402_1005Metric, F.Cu at (183.6, 86.0)
- added CL7: 100nF, Capacitor_SMD:C_0402_1005Metric, F.Cu at (202.8, 129.7)
- added CL8: 100nF, Capacitor_SMD:C_0402_1005Metric, F.Cu at (183.6, 173.3)
- added CL9: 100nF, Capacitor_SMD:C_0402_1005Metric, F.Cu at (68.4, 86.0)
- added CS1: 100nF, Capacitor_SMD:C_0402_1005Metric, F.Cu at (126.0, 109.8)
- added CS10: 100nF, Capacitor_SMD:C_0402_1005Metric, F.Cu at (202.8, 87.9)
- added CS11: 100nF, Capacitor_SMD:C_0402_1005Metric, F.Cu at (145.2, 153.5)
- added CS12: 100nF, Capacitor_SMD:C_0402_1005Metric, F.Cu at (106.8, 87.9)
- added CS13: 100nF, Capacitor_SMD:C_0402_1005Metric, F.Cu at (123.5, 56.1)
- added CS14: 100nF, Capacitor_SMD:C_0402_1005Metric, F.Cu at (145.2, 87.9)
- added CS15: 100nF, Capacitor_SMD:C_0402_1005Metric, F.Cu at (87.6, 131.6)
- added CS16: 100nF, Capacitor_SMD:C_0402_1005Metric, F.Cu at (68.4, 109.8)
- added CS17: 100nF, Capacitor_SMD:C_0402_1005Metric, F.Cu at (87.6, 153.5)
- added CS18: 100nF, Capacitor_SMD:C_0402_1005Metric, F.Cu at (106.8, 175.3)
- added CS19: 100nF, Capacitor_SMD:C_0402_1005Metric, F.Cu at (181.1, 56.1)
- added CS2: 100nF, Capacitor_SMD:C_0402_1005Metric, F.Cu at (68.4, 153.5)
- added CS20: 100nF, Capacitor_SMD:C_0402_1005Metric, F.Cu at (145.2, 175.3)
- added CS21: 100nF, Capacitor_SMD:C_0402_1005Metric, F.Cu at (106.8, 109.8)
- added CS22: 100nF, Capacitor_SMD:C_0402_1005Metric, F.Cu at (183.6, 153.5)
- added CS23: 100nF, Capacitor_SMD:C_0402_1005Metric, F.Cu at (164.4, 87.9)
- added CS24: 100nF, Capacitor_SMD:C_0402_1005Metric, F.Cu at (142.7, 56.1)
- added CS25: 100nF, Capacitor_SMD:C_0402_1005Metric, F.Cu at (87.6, 109.8)
- added CS26: 100nF, Capacitor_SMD:C_0402_1005Metric, F.Cu at (202.8, 109.8)
- added CS27: 100nF, Capacitor_SMD:C_0402_1005Metric, F.Cu at (126.0, 131.6)
- added CS28: 100nF, Capacitor_SMD:C_0402_1005Metric, F.Cu at (126.0, 87.9)
- added CS29: 100nF, Capacitor_SMD:C_0402_1005Metric, F.Cu at (145.2, 109.8)
- added CS3: 100nF, Capacitor_SMD:C_0402_1005Metric, F.Cu at (202.8, 153.5)
- added CS30: 100nF, Capacitor_SMD:C_0402_1005Metric, F.Cu at (161.9, 56.1)
- added CS31: 100nF, Capacitor_SMD:C_0402_1005Metric, F.Cu at (87.6, 175.3)
- added CS32: 100nF, Capacitor_SMD:C_0402_1005Metric, F.Cu at (145.2, 131.6)
- added CS33: 100nF, Capacitor_SMD:C_0402_1005Metric, F.Cu at (68.4, 175.3)
- added CS34: 100nF, Capacitor_SMD:C_0402_1005Metric, F.Cu at (126.0, 153.5)
- added CS35: 100nF, Capacitor_SMD:C_0402_1005Metric, F.Cu at (164.4, 153.5)
- added CS36: 100nF, Capacitor_SMD:C_0402_1005Metric, F.Cu at (183.6, 131.6)
- added CS37: 100nF, Capacitor_SMD:C_0402_1005Metric, F.Cu at (164.4, 131.6)
- added CS38: 100nF, Capacitor_SMD:C_0402_1005Metric, F.Cu at (87.6, 87.9)
- added CS39: 100nF, Capacitor_SMD:C_0402_1005Metric, F.Cu at (106.8, 153.5)
- added CS4: 100nF, Capacitor_SMD:C_0402_1005Metric, F.Cu at (183.6, 109.8)
- added CS40: 100nF, Capacitor_SMD:C_0402_1005Metric, F.Cu at (126.0, 175.3)
- added CS41: 100nF, Capacitor_SMD:C_0402_1005Metric, F.Cu at (68.4, 131.6)
- added CS43: 100nF, Capacitor_SMD:C_0402_1005Metric, F.Cu at (200.3, 56.1)
- added CS45: 100nF, Capacitor_SMD:C_0402_1005Metric, F.Cu at (164.4, 175.3)
- added CS46: 100nF, Capacitor_SMD:C_0402_1005Metric, F.Cu at (202.8, 175.3)
- added CS47: 100nF, Capacitor_SMD:C_0402_1005Metric, F.Cu at (106.8, 131.6)
- added CS5: 100nF, Capacitor_SMD:C_0402_1005Metric, F.Cu at (164.4, 109.8)
- added CS6: 100nF, Capacitor_SMD:C_0402_1005Metric, F.Cu at (183.6, 87.9)
- added CS7: 100nF, Capacitor_SMD:C_0402_1005Metric, F.Cu at (202.8, 131.6)
- added CS8: 100nF, Capacitor_SMD:C_0402_1005Metric, F.Cu at (183.6, 175.3)
- added CS9: 100nF, Capacitor_SMD:C_0402_1005Metric, F.Cu at (68.4, 87.9)
- added D1: Red, LED_SMD:LED_0603_1608Metric, F.Cu at (83.8, 50.7)
- added D2: Red, LED_SMD:LED_0603_1608Metric, F.Cu at (83.8, 53.3)
- added D3: 6V ESD, footprint:SOD-123FL_L2.8-W1.8-LS3.7-BI, F.Cu at (105.5, 48.5)
- added D6: Red, LED_SMD:LED_0603_1608Metric, F.Cu at (83.8, 55.9)
- added D7: 6V ESD, footprint:SOD-123FL_L2.8-W1.8-LS3.7-BI, F.Cu at (67.9, 65.4)
- added J1: Debug, Connector_PinHeader_2.54mm:PinHeader_1x04_P2.54mm_Vertical, F.Cu at (58.1, 52.6)
- added J2: I2C, Connector_PinHeader_2.54mm:PinHeader_1x04_P2.54mm_Vertical, F.Cu at (95.7, 39.9)
- added J3: ALS, Connector_PinHeader_2.54mm:PinHeader_1x03_P2.54mm_Vertical, F.Cu at (100.4, 49.2)
- added J4: Serial, Connector_PinHeader_2.54mm:PinHeader_1x05_P2.54mm_Vertical, F.Cu at (91.1, 39.9)
- added PB1: TS-1187A-B-A-B, footprint:SW-SMD_4P-L5.1-W5.1-P3.70-LS6.5-TL-2, F.Cu at (60.5, 40.8)
- added PB2: TS-1187A-B-A-B, footprint:SW-SMD_4P-L5.1-W5.1-P3.70-LS6.5-TL-2, F.Cu at (60.5, 47.1)
- added R1: 15k, Resistor_SMD:R_0402_1005Metric, F.Cu at (66.5, 50.4)
- added R10: 5.1k, Resistor_SMD:R_0402_1005Metric, F.Cu at (69.5, 52.4)
- added R11: 5.1k, Resistor_SMD:R_0402_1005Metric, F.Cu at (69.5, 54.4)
- added R12: 5.1k, Resistor_SMD:R_0402_1005Metric, F.Cu at (69.5, 56.4)
- added R13: 1.5k, Resistor_SMD:R_0402_1005Metric, F.Cu at (69.5, 58.4)
- added R2: 15k, Resistor_SMD:R_0402_1005Metric, F.Cu at (66.5, 52.4)
- added R3: 15k, Resistor_SMD:R_0402_1005Metric, F.Cu at (66.5, 54.4)
- added R4: 5.1k, Resistor_SMD:R_0402_1005Metric, F.Cu at (66.5, 56.4)
- added R5: 1.5k, Resistor_SMD:R_0402_1005Metric, F.Cu at (66.5, 58.4)
- added R9: 5.1k, Resistor_SMD:R_0402_1005Metric, F.Cu at (69.5, 50.4)
- added RA10: 68kΩ, footprint:R0402, F.Cu at (199.9, 86.1)
- added RA11: 68kΩ, footprint:R0402, F.Cu at (142.3, 151.6)
- added RA12: 68kΩ, footprint:R0402, F.Cu at (103.8, 86.1)
- added RA13: 68kΩ, footprint:R0402, F.Cu at (120.5, 54.2)
- added RA14: 68kΩ, footprint:R0402, F.Cu at (142.3, 86.1)
- added RA15: 68kΩ, footprint:R0402, F.Cu at (84.6, 129.7)
- added RA16: 68kΩ, footprint:R0402, F.Cu at (65.4, 107.9)
- added RA17: 68kΩ, footprint:R0402, F.Cu at (84.6, 151.6)
- added RA18: 68kΩ, footprint:R0402, F.Cu at (103.8, 173.4)
- added RA19: 68kΩ, footprint:R0402, F.Cu at (178.2, 54.2)
- added RA20: 68kΩ, footprint:R0402, F.Cu at (142.3, 173.4)
- added RA21: 68kΩ, footprint:R0402, F.Cu at (103.8, 107.9)
- added RA22: 68kΩ, footprint:R0402, F.Cu at (180.7, 151.6)
- added RA23: 68kΩ, footprint:R0402, F.Cu at (161.5, 86.1)
- added RA24: 68kΩ, footprint:R0402, F.Cu at (139.7, 54.2)
- added RA25: 68kΩ, footprint:R0402, F.Cu at (84.6, 107.9)
- added RA26: 68kΩ, footprint:R0402, F.Cu at (199.9, 107.9)
- added RA27: 68kΩ, footprint:R0402, F.Cu at (123.1, 129.7)
- added RA28: 68kΩ, footprint:R0402, F.Cu at (123.1, 86.1)
- added RA29: 68kΩ, footprint:R0402, F.Cu at (142.3, 107.9)
- added RA30: 68kΩ, footprint:R0402, F.Cu at (158.9, 54.2)
- added RA31: 68kΩ, footprint:R0402, F.Cu at (84.6, 173.4)
- added RA32: 68kΩ, footprint:R0402, F.Cu at (142.3, 129.7)
- added RA33: 68kΩ, footprint:R0402, F.Cu at (65.4, 173.4)
- added RA34: 68kΩ, footprint:R0402, F.Cu at (123.1, 151.6)
- added RA35: 68kΩ, footprint:R0402, F.Cu at (161.5, 151.6)
- added RA36: 68kΩ, footprint:R0402, F.Cu at (180.7, 129.7)
- added RA37: 68kΩ, footprint:R0402, F.Cu at (161.5, 129.7)
- added RA38: 68kΩ, footprint:R0402, F.Cu at (84.6, 86.1)
- added RA39: 68kΩ, footprint:R0402, F.Cu at (103.8, 151.6)
- added RA40: 68kΩ, footprint:R0402, F.Cu at (123.1, 173.4)
- added RA41: 68kΩ, footprint:R0402, F.Cu at (65.4, 129.7)
- added RA43: 68kΩ, footprint:R0402, F.Cu at (197.4, 54.2)
- added RA45: 68kΩ, footprint:R0402, F.Cu at (161.5, 173.4)
- added RA46: 68kΩ, footprint:R0402, F.Cu at (199.9, 173.4)
- added RA47: 68kΩ, footprint:R0402, F.Cu at (103.8, 129.7)
- added RA9: 68kΩ, footprint:R0402, F.Cu at (65.4, 86.1)
- added RB10: 33kΩ, footprint:R0402, F.Cu at (199.9, 88.2)
- added RB11: 33kΩ, footprint:R0402, F.Cu at (142.3, 153.7)
- added RB12: 33kΩ, footprint:R0402, F.Cu at (103.8, 88.2)
- added RB13: 33kΩ, footprint:R0402, F.Cu at (120.5, 56.3)
- added RB14: 33kΩ, footprint:R0402, F.Cu at (142.3, 88.2)
- added RB15: 33kΩ, footprint:R0402, F.Cu at (84.6, 131.9)
- added RB16: 33kΩ, footprint:R0402, F.Cu at (65.4, 110.0)
- added RB17: 33kΩ, footprint:R0402, F.Cu at (84.6, 153.7)
- added RB18: 33kΩ, footprint:R0402, F.Cu at (103.8, 175.6)
- added RB19: 33kΩ, footprint:R0402, F.Cu at (178.2, 56.3)
- added RB20: 33kΩ, footprint:R0402, F.Cu at (142.3, 175.6)
- added RB21: 33kΩ, footprint:R0402, F.Cu at (103.8, 110.0)
- added RB22: 33kΩ, footprint:R0402, F.Cu at (180.7, 153.7)
- added RB23: 33kΩ, footprint:R0402, F.Cu at (161.5, 88.2)
- added RB24: 33kΩ, footprint:R0402, F.Cu at (139.7, 56.3)
- added RB25: 33kΩ, footprint:R0402, F.Cu at (84.6, 110.0)
- added RB26: 33kΩ, footprint:R0402, F.Cu at (199.9, 110.0)
- added RB27: 33kΩ, footprint:R0402, F.Cu at (123.1, 131.9)
- added RB28: 33kΩ, footprint:R0402, F.Cu at (123.1, 88.2)
- added RB29: 33kΩ, footprint:R0402, F.Cu at (142.3, 110.0)
- added RB30: 33kΩ, footprint:R0402, F.Cu at (158.9, 56.3)
- added RB31: 33kΩ, footprint:R0402, F.Cu at (84.6, 175.6)
- added RB32: 33kΩ, footprint:R0402, F.Cu at (142.3, 131.9)
- added RB33: 33kΩ, footprint:R0402, F.Cu at (65.4, 175.6)
- added RB34: 33kΩ, footprint:R0402, F.Cu at (123.1, 153.7)
- added RB35: 33kΩ, footprint:R0402, F.Cu at (161.5, 153.7)
- added RB36: 33kΩ, footprint:R0402, F.Cu at (180.7, 131.9)
- added RB37: 33kΩ, footprint:R0402, F.Cu at (161.5, 131.9)
- added RB38: 33kΩ, footprint:R0402, F.Cu at (84.6, 88.2)
- added RB39: 33kΩ, footprint:R0402, F.Cu at (103.8, 153.7)
- added RB40: 33kΩ, footprint:R0402, F.Cu at (123.1, 175.6)
- added RB41: 33kΩ, footprint:R0402, F.Cu at (65.4, 131.9)
- added RB43: 33kΩ, footprint:R0402, F.Cu at (197.4, 56.3)
- added RB45: 33kΩ, footprint:R0402, F.Cu at (161.5, 175.6)
- added RB46: 33kΩ, footprint:R0402, F.Cu at (199.9, 175.6)
- added RB47: 33kΩ, footprint:R0402, F.Cu at (103.8, 131.9)
- added RB9: 33kΩ, footprint:R0402, F.Cu at (65.4, 88.2)
- added SR2: 74HC165, Package_SO:SOIC-16_3.9x9.9mm_P1.27mm, F.Cu at (175.3, 184.4)
- added SR3: 74HC165, Package_SO:SOIC-16_3.9x9.9mm_P1.27mm, F.Cu at (156.1, 184.4)
- added SR4: 74HC165, Package_SO:SOIC-16_3.9x9.9mm_P1.27mm, F.Cu at (194.5, 184.4)
- added SR5: 74HC165, Package_SO:SOIC-16_3.9x9.9mm_P1.27mm, F.Cu at (136.9, 184.4)
- added SR6: 74HC165, Package_SO:SOIC-16_3.9x9.9mm_P1.27mm, F.Cu at (98.4, 184.4)
- added STM1: STM32F103C8Tx, Package_QFP:LQFP-48_7x7mm_P0.5mm, F.Cu at (76.5, 43.2)
- added SW10: SW_Push, PCM_Switch_Keyboard_Hotswap_Kailh:SW_Hotswap_Kailh_MX, F.Cu at (199.1, 77.2)
- added SW11: SW_Push, PCM_Switch_Keyboard_Hotswap_Kailh:SW_Hotswap_Kailh_MX, F.Cu at (141.5, 142.7)
- added SW12: SW_Push, PCM_Switch_Keyboard_Hotswap_Kailh:SW_Hotswap_Kailh_MX, F.Cu at (103.1, 77.2)
- added SW13: SW_Push, PCM_Switch_Keyboard_Hotswap_Kailh:SW_Hotswap_Kailh_MX, F.Cu at (119.8, 45.4)
- added SW14: SW_Push, PCM_Switch_Keyboard_Hotswap_Kailh:SW_Hotswap_Kailh_MX, F.Cu at (141.5, 77.2)
- added SW15: SW_Push, PCM_Switch_Keyboard_Hotswap_Kailh:SW_Hotswap_Kailh_MX, F.Cu at (83.9, 120.9)
- added SW16: SW_Push, PCM_Switch_Keyboard_Hotswap_Kailh:SW_Hotswap_Kailh_MX, F.Cu at (64.7, 99.0)
- added SW17: SW_Push, PCM_Switch_Keyboard_Hotswap_Kailh:SW_Hotswap_Kailh_MX, F.Cu at (83.9, 142.7)
- added SW18: SW_Push, PCM_Switch_Keyboard_Hotswap_Kailh:SW_Hotswap_Kailh_MX, F.Cu at (103.1, 164.6)
- added SW19: SW_Push, PCM_Switch_Keyboard_Hotswap_Kailh:SW_Hotswap_Kailh_MX, F.Cu at (177.4, 45.4)
- added SW20: SW_Push, PCM_Switch_Keyboard_Hotswap_Kailh:SW_Hotswap_Kailh_MX, F.Cu at (141.5, 164.6)
- added SW21: SW_Push, PCM_Switch_Keyboard_Hotswap_Kailh:SW_Hotswap_Kailh_MX, F.Cu at (103.1, 99.0)
- added SW22: SW_Push, PCM_Switch_Keyboard_Hotswap_Kailh:SW_Hotswap_Kailh_MX, F.Cu at (179.9, 142.7)
- added SW23: SW_Push, PCM_Switch_Keyboard_Hotswap_Kailh:SW_Hotswap_Kailh_MX, F.Cu at (160.7, 77.2)
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Connections:
- C1 pad 2: /Key Column/SW1 -> Net-(STM1-PD0)
- C2 pad 2: /Key Column/SW2 -> Net-(STM1-PD1)
- C3 pad 2: /Key Column/SW3 -> +3.3V
- C4 pad 2: /Key Column/SW4 -> +3.3V
- C5 pad 2: /Key Column/SW5 -> +3.3V
- C6 pad 2: /Key Column/SW6 -> +3.3V
- C7 pad 2: /Key Column/SW7 -> +3.3V
- C8 pad 2: /Key Column/SW8 -> +3.3V
- RB1 pad 1: /Key Column/SW1 -> /Left Half/8-Key Module1/Key Unit7/SwitchOutput
- RB2 pad 1: /Key Column/SW2 -> /Left Half/8-Key Module4/Key Unit3/SwitchOutput
- RB3 pad 1: /Key Column/SW3 -> /Left Half/8-Key Module/Key Unit2/SwitchOutput
- RB4 pad 1: /Key Column/SW4 -> /Left Half/8-Key Module2/Key Unit6/SwitchOutput
- RB5 pad 1: /Key Column/SW5 -> /Left Half/8-Key Module2/Key Unit0/SwitchOutput
- RB6 pad 1: /Key Column/SW6 -> /Left Half/8-Key Module1/Key Unit0/SwitchOutput
- RB7 pad 1: /Key Column/SW7 -> /Left Half/5-Key Module/Key Unit8/SwitchOutput
- RB8 pad 1: /Key Column/SW8 -> /Left Half/8-Key Module/Key Unit1/SwitchOutput
- SR1 pad 1: unconnected-(SR1-~{PL}-Pad1) -> /Left Half/5-Key Module/SR_LOAD
- SR1 pad 10: unconnected-(SR1-DS-Pad10) -> /Left Half/8-Key Module1/SR_OUT
- SR1 pad 11: /Key Column/SW1 -> /Left Half/8-Key Module2/Key Unit7/SwitchOutput
- SR1 pad 12: /Key Column/SW2 -> /Left Half/8-Key Module2/Key Unit6/SwitchOutput
- SR1 pad 13: /Key Column/SW3 -> /Left Half/8-Key Module2/Key Unit5/SwitchOutput
- SR1 pad 14: /Key Column/SW4 -> /Left Half/8-Key Module2/Key Unit4/SwitchOutput
- SR1 pad 2: unconnected-(SR1-CP-Pad2) -> /Left Half/5-Key Module/SR_CLOCK
- SR1 pad 3: /Key Column/SW5 -> /Left Half/8-Key Module2/Key Unit3/SwitchOutput
- SR1 pad 4: /Key Column/SW6 -> /Left Half/8-Key Module2/Key Unit2/SwitchOutput
- SR1 pad 5: /Key Column/SW7 -> /Left Half/8-Key Module2/Key Unit1/SwitchOutput
- SR1 pad 6: /Key Column/SW8 -> /Left Half/8-Key Module2/Key Unit0/SwitchOutput
- SR1 pad 9: unconnected-(SR1-Q7-Pad9) -> /Left Half/8-Key Module2/SR_OUT

Commit message: Plugin works.
Parts:
- removed C1, C2: 30pF, Capacitor_SMD:C_0402_1005Metric
- removed C10: 4.7uF, Capacitor_SMD:C_0603_1608Metric
- removed C11, C12, C3, C4, C5, C6, C8, CL1, CL10, CL11, CL12, CL13, CL14, CL15, CL16, CL17, CL18, CL19, CL2, CL20, CL21, CL22, CL23, CL24, CL25, CL26, CL27, CL28, CL29, CL3, CL30, CL31, CL32, CL33, CL34, CL35, CL36, CL37, CL38, CL39, CL4, CL40, CL41, CL43, CL45, CL46, CL47, CL5, CL6, CL7, CL8, CL9, CS1, CS10, CS11, CS12, CS13, CS14, CS15, CS16, CS17, CS18, CS19, CS2, CS20, CS21, CS22, CS23, CS24, CS25, CS26, CS27, CS28, CS29, CS3, CS30, CS31, CS32, CS33, CS34, CS35, CS36, CS37, CS38, CS39, CS4, CS40, CS41, CS43, CS45, CS46, CS47, CS5, CS6, CS7, CS8, CS9: 100nF, Capacitor_SMD:C_0402_1005Metric
- removed C13, C14: 100uF, Capacitor_Tantalum_SMD:CP_EIA-3528-15_AVX-H
- removed C7: 10nF, Capacitor_SMD:C_0402_1005Metric
- removed C9: 1uF, Capacitor_SMD:C_0402_1005Metric
- removed D1, D2, D6: Red, LED_SMD:LED_0603_1608Metric
- removed D3, D7: 6V ESD, footprint:SOD-123FL_L2.8-W1.8-LS3.7-BI
- removed J1: Debug, Connector_PinHeader_2.54mm:PinHeader_1x04_P2.54mm_Vertical
- removed J2: I2C, Connector_PinHeader_2.54mm:PinHeader_1x04_P2.54mm_Vertical
- removed J3: ALS, Connector_PinHeader_2.54mm:PinHeader_1x03_P2.54mm_Vertical
- removed J4: Serial, Connector_PinHeader_2.54mm:PinHeader_1x05_P2.54mm_Vertical
- removed PB1, PB2: TS-1187A-B-A-B, footprint:SW-SMD_4P-L5.1-W5.1-P3.70-LS6.5-TL-2
- removed R1, R2, R3: 15k, Resistor_SMD:R_0402_1005Metric
- removed R10, R11, R12, R4, R9: 5.1k, Resistor_SMD:R_0402_1005Metric
- removed R13, R5: 1.5k, Resistor_SMD:R_0402_1005Metric
- removed RA1, RA10, RA11, RA12, RA13, RA14, RA15, RA16, RA17, RA18, RA19, RA2, RA20, RA21, RA22, RA23, RA24, RA25, RA26, RA27, RA28, RA29, RA3, RA30, RA31, RA32, RA33, RA34, RA35, RA36, RA37, RA38, RA39, RA4, RA40, RA41, RA43, RA45, RA46, RA47, RA5, RA6, RA7, RA8, RA9: 68kΩ, footprint:R0402
- removed RB1, RB10, RB11, RB12, RB13, RB14, RB15, RB16, RB17, RB18, RB19, RB2, RB20, RB21, RB22, RB23, RB24, RB25, RB26, RB27, RB28, RB29, RB3, RB30, RB31, RB32, RB33, RB34, RB35, RB36, RB37, RB38, RB39, RB4, RB40, RB41, RB43, RB45, RB46, RB47, RB5, RB6, RB7, RB8, RB9: 33kΩ, footprint:R0402
- removed SR1, SR2, SR3, SR4, SR5, SR6: 74HC165, Package_SO:SOIC-16_3.9x9.9mm_P1.27mm
- removed STM1: STM32F103C8Tx, Package_QFP:LQFP-48_7x7mm_P0.5mm
- removed SW1, SW10, SW11, SW12, SW13, SW14, SW15, SW16, SW17, SW18, SW19, SW2, SW20, SW21, SW22, SW23, SW24, SW25, SW26, SW27, SW28, SW29, SW3, SW30, SW31, SW32, SW33, SW34, SW35, SW36, SW37, SW38, SW39, SW4, SW40, SW41, SW43, SW45, SW46, SW47, SW5, SW6, SW7, SW8, SW9: SW_Push, PCM_Switch_Keyboard_Hotswap_Kailh:SW_Hotswap_Kailh_MX
- removed U1, U10, U11, U12, U13, U14, U15, U16, U17, U18, U19, U2, U20, U21, U22, U23, U24, U25, U26, U27, U28, U29, U3, U30, U31, U32, U33, U34, U35, U36, U37, U38, U39, U4, U40, U41, U43, U45, U46, U47, U5, U6, U7, U8, U9: SK6812MINI-E_C5149201, footprint:LED-SMD_L3.2-W2.8-TR
- removed U42: AMS1117-3.3, Package_TO_SOT_SMD:SOT-223-3_TabPin2
- removed U44, U49: TYPE-C-31-M-12, footprint:USB-C_SMD-TYPE-C-31-M-12
- removed U48, U50: USBLC6-2SC6, Package_TO_SOT_SMD:SOT-23-6
- removed X1: Crystal, Crystal:Crystal_SMD_3225-4Pin_3.2x2.5mm
- added C55001: 30pF, Capacitor_SMD:C_0402_1005Metric, F.Cu at (-21.7, -17.9)
- added C55002: 30pF, Capacitor_SMD:C_0402_1005Metric, F.Cu at (-21.7, -15.9)
- added C55003: 100nF, Capacitor_SMD:C_0402_1005Metric, F.Cu at (-21.7, -13.9)
- added C55004: 100nF, Capacitor_SMD:C_0402_1005Metric, F.Cu at (-21.7, -12.0)
- added C55005: 100nF, Capacitor_SMD:C_0402_1005Metric, F.Cu at (-21.7, -10.00)
- added C55006: 100nF, Capacitor_SMD:C_0402_1005Metric, F.Cu at (-21.7, -8.03)
- added C55007: 10nF, Capacitor_SMD:C_0402_1005Metric, F.Cu at (-18.8, -17.9)
- added C55008: 100nF, Capacitor_SMD:C_0402_1005Metric, F.Cu at (-18.8, -15.9)
- added C55009: 1uF, Capacitor_SMD:C_0402_1005Metric, F.Cu at (-18.8, -13.9)
- added C55010: 4.7uF, Capacitor_SMD:C_0603_1608Metric, F.Cu at (-25.2, 7.34)
- added C55011: 100nF, Capacitor_SMD:C_0402_1005Metric, F.Cu at (-18.8, -12.0)
- added C55012: 100nF, Capacitor_SMD:C_0402_1005Metric, F.Cu at (-18.8, -10.00)
- added C55013: 100uF, Capacitor_Tantalum_SMD:CP_EIA-3528-15_AVX-H, F.Cu at (-14.3, 4.47)
- added C55014: 100uF, Capacitor_Tantalum_SMD:CP_EIA-3528-15_AVX-H, F.Cu at (-14.3, 8.82)
- added CL10001: 100nF, Capacitor_SMD:C_0402_1005Metric, B.Cu at (164.3, 149.2)
- added CL11001: 100nF, Capacitor_SMD:C_0402_1005Metric, B.Cu at (145.1, 127.4)
- added CL12001: 100nF, Capacitor_SMD:C_0402_1005Metric, B.Cu at (183.5, 40.0)
- added CL13001: 100nF, Capacitor_SMD:C_0402_1005Metric, B.Cu at (221.9, 18.2)
- added CL14001: 100nF, Capacitor_SMD:C_0402_1005Metric, B.Cu at (30.6, 62.5)
- added CL17001: 100nF, Capacitor_SMD:C_0402_1005Metric, B.Cu at (183.5, 127.4)
- added CL18001: 100nF, Capacitor_SMD:C_0402_1005Metric, B.Cu at (221.9, 83.7)
- added CL19001: 100nF, Capacitor_SMD:C_0402_1005Metric, B.Cu at (145.1, 149.2)
- added CL20001: 100nF, Capacitor_SMD:C_0402_1005Metric, B.Cu at (221.9, 61.8)
- added CL2001: 100nF, Capacitor_SMD:C_0402_1005Metric, B.Cu at (202.7, 61.8)
- added CL21001: 100nF, Capacitor_SMD:C_0402_1005Metric, B.Cu at (164.3, 105.5)
- added CL22001: 100nF, Capacitor_SMD:C_0402_1005Metric, B.Cu at (183.5, 149.2)
- added CL23001: 100nF, Capacitor_SMD:C_0402_1005Metric, B.Cu at (183.5, 18.2)
- added CL24001: 100nF, Capacitor_SMD:C_0402_1005Metric, B.Cu at (125.9, 127.4)
- added CL25001: 100nF, Capacitor_SMD:C_0402_1005Metric, B.Cu at (164.3, 40.0)
- added CL26001: 100nF, Capacitor_SMD:C_0402_1005Metric, B.Cu at (202.7, 83.7)
- added CL27001: 100nF, Capacitor_SMD:C_0402_1005Metric, B.Cu at (221.9, 149.2)
- added CL28001: 100nF, Capacitor_SMD:C_0402_1005Metric, B.Cu at (221.9, 105.5)
- added CL30001: 100nF, Capacitor_SMD:C_0402_1005Metric, B.Cu at (145.1, 105.5)
- added CL3001: 100nF, Capacitor_SMD:C_0402_1005Metric, B.Cu at (106.6, 149.2)
- added CL31001: 100nF, Capacitor_SMD:C_0402_1005Metric, B.Cu at (125.9, 105.5)
- added CL33001: 100nF, Capacitor_SMD:C_0402_1005Metric, B.Cu at (202.7, 127.4)
- added CL34001: 100nF, Capacitor_SMD:C_0402_1005Metric, B.Cu at (202.7, 40.0)
- added CL35001: 100nF, Capacitor_SMD:C_0402_1005Metric, B.Cu at (202.7, 149.2)
- added CL36001: 100nF, Capacitor_SMD:C_0402_1005Metric, B.Cu at (221.9, 40.0)
- added CL37001: 100nF, Capacitor_SMD:C_0402_1005Metric, B.Cu at (183.5, 61.8)
- added CL38001: 100nF, Capacitor_SMD:C_0402_1005Metric, B.Cu at (145.1, 40.0)
- added CL39001: 100nF, Capacitor_SMD:C_0402_1005Metric, B.Cu at (106.6, 105.5)
- added CL40001: 100nF, Capacitor_SMD:C_0402_1005Metric, B.Cu at (106.6, 83.7)
- added CL4001: 100nF, Capacitor_SMD:C_0402_1005Metric, B.Cu at (164.3, 18.2)
- added CL41001: 100nF, Capacitor_SMD:C_0402_1005Metric, B.Cu at (145.1, 83.7)
- added CL43001: 100nF, Capacitor_SMD:C_0402_1005Metric, B.Cu at (164.3, 83.7)
- added CL44001: 100nF, Capacitor_SMD:C_0402_1005Metric, B.Cu at (223.8, 126.7)
- added CL45001: 100nF, Capacitor_SMD:C_0402_1005Metric, B.Cu at (202.7, 105.5)
- added CL46001: 100nF, Capacitor_SMD:C_0402_1005Metric, B.Cu at (183.5, 83.7)
- added CL47001: 100nF, Capacitor_SMD:C_0402_1005Metric, B.Cu at (125.9, 149.2)
- added CL48001: 100nF, Capacitor_SMD:C_0402_1005Metric, B.Cu at (28.9, 115.7)
- added CL50001: 100nF, Capacitor_SMD:C_0402_1005Metric, B.Cu at (164.3, 61.8)
- added CL5001: 100nF, Capacitor_SMD:C_0402_1005Metric, B.Cu at (183.5, 105.5)
- added CL51001: 100nF, Capacitor_SMD:C_0402_1005Metric, B.Cu at (51.9, 54.3)
- added CL52001: 100nF, Capacitor_SMD:C_0402_1005Metric, B.Cu at (79.9, 58.4)
- added CL53001: 100nF, Capacitor_SMD:C_0402_1005Metric, B.Cu at (106.6, 127.4)
- added CL56001: 100nF, Capacitor_SMD:C_0402_1005Metric, B.Cu at (-51.1, 68.3)
- added CL57001: 100nF, Capacitor_SMD:C_0402_1005Metric, B.Cu at (-31.9, 68.3)
- added CL58001: 100nF, Capacitor_SMD:C_0402_1005Metric, B.Cu at (-31.9, 46.5)
- added CL59001: 100nF, Capacitor_SMD:C_0402_1005Metric, B.Cu at (-51.1, 46.5)
- added CL6001: 100nF, Capacitor_SMD:C_0402_1005Metric, B.Cu at (202.7, 18.2)
- added CL7001: 100nF, Capacitor_SMD:C_0402_1005Metric, B.Cu at (164.3, 127.4)
- added CL8001: 100nF, Capacitor_SMD:C_0402_1005Metric, B.Cu at (125.9, 83.7)
- added CL9001: 100nF, Capacitor_SMD:C_0402_1005Metric, B.Cu at (145.1, 61.8)
- added CS10001: 100nF, Capacitor_SMD:C_0402_1005Metric, B.Cu at (167.5, 147.6)
- added CS11001: 100nF, Capacitor_SMD:C_0402_1005Metric, B.Cu at (148.3, 125.8)
- added CS12001: 100nF, Capacitor_SMD:C_0402_1005Metric, B.Cu at (186.7, 38.4)
- added CS13001: 100nF, Capacitor_SMD:C_0402_1005Metric, B.Cu at (225.1, 16.6)
- added CS14001: 100nF, Capacitor_SMD:C_0402_1005Metric, B.Cu at (33.0, 59.9)
- added CS17001: 100nF, Capacitor_SMD:C_0402_1005Metric, B.Cu at (186.7, 125.8)
- added CS18001: 100nF, Capacitor_SMD:C_0402_1005Metric, B.Cu at (225.1, 82.1)
- added CS19001: 100nF, Capacitor_SMD:C_0402_1005Metric, B.Cu at (148.3, 147.6)
- added CS20001: 100nF, Capacitor_SMD:C_0402_1005Metric, B.Cu at (225.1, 60.2)
- added CS2001: 100nF, Capacitor_SMD:C_0402_1005Metric, B.Cu at (205.9, 60.2)
- added CS21001: 100nF, Capacitor_SMD:C_0402_1005Metric, B.Cu at (167.5, 103.9)
- added CS22001: 100nF, Capacitor_SMD:C_0402_1005Metric, B.Cu at (186.7, 147.6)
- added CS23001: 100nF, Capacitor_SMD:C_0402_1005Metric, B.Cu at (186.7, 16.6)
- added CS24001: 100nF, Capacitor_SMD:C_0402_1005Metric, B.Cu at (129.1, 125.8)
- added CS25001: 100nF, Capacitor_SMD:C_0402_1005Metric, B.Cu at (167.5, 38.4)
- added CS26001: 100nF, Capacitor_SMD:C_0402_1005Metric, B.Cu at (205.9, 82.1)
- added CS27001: 100nF, Capacitor_SMD:C_0402_1005Metric, B.Cu at (225.1, 147.6)
- added CS28001: 100nF, Capacitor_SMD:C_0402_1005Metric, B.Cu at (225.1, 103.9)
- added CS30001: 100nF, Capacitor_SMD:C_0402_1005Metric, B.Cu at (148.3, 103.9)
- added CS3001: 100nF, Capacitor_SMD:C_0402_1005Metric, B.Cu at (109.8, 147.6)
- added CS31001: 100nF, Capacitor_SMD:C_0402_1005Metric, B.Cu at (129.1, 103.9)
- added CS33001: 100nF, Capacitor_SMD:C_0402_1005Metric, B.Cu at (205.9, 125.8)
- added CS34001: 100nF, Capacitor_SMD:C_0402_1005Metric, B.Cu at (205.9, 38.4)
- added CS35001: 100nF, Capacitor_SMD:C_0402_1005Metric, B.Cu at (205.9, 147.6)
- added CS36001: 100nF, Capacitor_SMD:C_0402_1005Metric, B.Cu at (225.1, 38.4)
- added CS37001: 100nF, Capacitor_SMD:C_0402_1005Metric, B.Cu at (186.7, 60.2)
- added CS38001: 100nF, Capacitor_SMD:C_0402_1005Metric, B.Cu at (148.3, 38.4)
- added CS39001: 100nF, Capacitor_SMD:C_0402_1005Metric, B.Cu at (109.8, 103.9)
- added CS40001: 100nF, Capacitor_SMD:C_0402_1005Metric, B.Cu at (109.8, 82.1)
- added CS4001: 100nF, Capacitor_SMD:C_0402_1005Metric, B.Cu at (167.5, 16.6)
- added CS41001: 100nF, Capacitor_SMD:C_0402_1005Metric, B.Cu at (148.3, 82.1)
- added CS43001: 100nF, Capacitor_SMD:C_0402_1005Metric, B.Cu at (167.5, 82.1)
- added CS44001: 100nF, Capacitor_SMD:C_0402_1005Metric, B.Cu at (227.0, 125.1)
- added CS45001: 100nF, Capacitor_SMD:C_0402_1005Metric, B.Cu at (205.9, 103.9)
- added CS46001: 100nF, Capacitor_SMD:C_0402_1005Metric, B.Cu at (186.7, 82.1)
- added CS47001: 100nF, Capacitor_SMD:C_0402_1005Metric, B.Cu at (129.1, 147.6)
- added CS48001: 100nF, Capacitor_SMD:C_0402_1005Metric, B.Cu at (32.1, 114.1)
- added CS50001: 100nF, Capacitor_SMD:C_0402_1005Metric, B.Cu at (167.5, 60.2)
- added CS5001: 100nF, Capacitor_SMD:C_0402_1005Metric, B.Cu at (186.7, 103.9)
- added CS51001: 100nF, Capacitor_SMD:C_0402_1005Metric, B.Cu at (54.8, 52.1)
- added CS52001: 100nF, Capacitor_SMD:C_0402_1005Metric, B.Cu at (83.5, 58.0)
- added CS53001: 100nF, Capacitor_SMD:C_0402_1005Metric, B.Cu at (109.8, 125.8)
- added CS56001: 100nF, Capacitor_SMD:C_0402_1005Metric, B.Cu at (-54.3, 69.9)
- added CS57001: 100nF, Capacitor_SMD:C_0402_1005Metric, B.Cu at (-35.1, 69.9)
- added CS58001: 100nF, Capacitor_SMD:C_0402_1005Metric, B.Cu at (-35.1, 48.1)
- added CS59001: 100nF, Capacitor_SMD:C_0402_1005Metric, B.Cu at (-54.3, 48.1)
- added CS6001: 100nF, Capacitor_SMD:C_0402_1005Metric, B.Cu at (205.9, 16.6)
- added CS7001: 100nF, Capacitor_SMD:C_0402_1005Metric, B.Cu at (167.5, 125.8)
- added CS8001: 100nF, Capacitor_SMD:C_0402_1005Metric, B.Cu at (129.1, 82.1)
- added CS9001: 100nF, Capacitor_SMD:C_0402_1005Metric, B.Cu at (148.3, 60.2)
- added D55001: Red, LED_SMD:LED_0603_1608Metric, F.Cu at (-4.43, -5.75)
- added D55002: 6V ESD, footprint:SOD-123FL_L2.8-W1.8-LS3.7-BI, F.Cu at (-20.3, 8.98)
- added D55003: Red, LED_SMD:LED_0603_1608Metric, F.Cu at (-4.43, -3.16)
- added D55004: Red, LED_SMD:LED_0603_1608Metric, F.Cu at (-4.43, -0.57)
- added D60001: 6V ESD, footprint:SOD-123FL_L2.8-W1.8-LS3.7-BI, F.Cu at (17.3, -7.90)
- added J55001: Debug, Connector_PinHeader_2.54mm:PinHeader_1x04_P2.54mm_Vertical, F.Cu at (-30.1, -3.84)
- added J60001: ALS, Connector_PinHeader_2.54mm:PinHeader_1x03_P2.54mm_Vertical, F.Cu at (12.1, -7.20)
- added J60002: Serial, Connector_PinHeader_2.54mm:PinHeader_1x05_P2.54mm_Vertical, F.Cu at (2.84, -16.5)
- added J60003: I2C, Connector_PinHeader_2.54mm:PinHeader_1x04_P2.54mm_Vertical, F.Cu at (7.49, -16.5)
- added PB55001: TS-1187A-B-A-B, footprint:SW-SMD_4P-L5.1-W5.1-P3.70-LS6.5-TL-2, F.Cu at (-27.8, -15.7)
- added PB55002: TS-1187A-B-A-B, footprint:SW-SMD_4P-L5.1-W5.1-P3.70-LS6.5-TL-2, F.Cu at (-27.8, -9.33)
- added R55001: 15k, Resistor_SMD:R_0402_1005Metric, F.Cu at (-21.7, -6.05)
- added R55002: 1.5k, Resistor_SMD:R_0402_1005Metric, F.Cu at (-21.7, -4.06)
- added R55003: 15k, Resistor_SMD:R_0402_1005Metric, F.Cu at (-21.7, -2.07)
- added R55004: 15k, Resistor_SMD:R_0402_1005Metric, F.Cu at (-21.7, -0.08)
- added R55005: 5.1k, Resistor_SMD:R_0402_1005Metric, F.Cu at (-21.7, 1.91)
- added R55006: 5.1k, Resistor_SMD:R_0402_1005Metric, F.Cu at (-18.8, -6.05)
- added R55007: 5.1k, Resistor_SMD:R_0402_1005Metric, F.Cu at (-18.8, -4.06)
- added R55008: 5.1k, Resistor_SMD:R_0402_1005Metric, F.Cu at (-18.8, -2.07)
- added R55009: 5.1k, Resistor_SMD:R_0402_1005Metric, F.Cu at (-18.8, -0.08)
- added R55010: 1.5k, Resistor_SMD:R_0402_1005Metric, F.Cu at (-18.8, 1.91)
- added RA10001: 68kΩ, footprint:R0402, B.Cu at (165.7, 149.2)
- added RA11001: 68kΩ, footprint:R0402, B.Cu at (146.5, 127.4)
- added RA12001: 68kΩ, footprint:R0402, B.Cu at (184.9, 40.0)
- added RA13001: 68kΩ, footprint:R0402, B.Cu at (223.3, 18.2)
- added RA14001: 68kΩ, footprint:R0402, B.Cu at (31.9, 62.1)
- added RA17001: 68kΩ, footprint:R0402, B.Cu at (184.9, 127.4)
- added RA18001: 68kΩ, footprint:R0402, B.Cu at (223.3, 83.7)
- added RA19001: 68kΩ, footprint:R0402, B.Cu at (146.5, 149.2)
- added RA20001: 68kΩ, footprint:R0402, B.Cu at (223.3, 61.8)
- added RA2001: 68kΩ, footprint:R0402, B.Cu at (204.1, 61.8)
- added RA21001: 68kΩ, footprint:R0402, B.Cu at (165.7, 105.5)
- added RA22001: 68kΩ, footprint:R0402, B.Cu at (184.9, 149.2)
- added RA23001: 68kΩ, footprint:R0402, B.Cu at (184.9, 18.2)
- added RA24001: 68kΩ, footprint:R0402, B.Cu at (127.3, 127.4)
- added RA25001: 68kΩ, footprint:R0402, B.Cu at (165.7, 40.0)
- added RA26001: 68kΩ, footprint:R0402, B.Cu at (204.1, 83.7)
- added RA27001: 68kΩ, footprint:R0402, B.Cu at (223.3, 149.2)
- added RA28001: 68kΩ, footprint:R0402, B.Cu at (223.3, 105.5)
- added RA30001: 68kΩ, footprint:R0402, B.Cu at (146.5, 105.5)
- added RA3001: 68kΩ, footprint:R0402, B.Cu at (108.0, 149.2)
- added RA31001: 68kΩ, footprint:R0402, B.Cu at (127.3, 105.5)
- added RA33001: 68kΩ, footprint:R0402, B.Cu at (204.1, 127.4)
- added RA34001: 68kΩ, footprint:R0402, B.Cu at (204.1, 40.0)
- added RA35001: 68kΩ, footprint:R0402, B.Cu at (204.1, 149.2)
- added RA36001: 68kΩ, footprint:R0402, B.Cu at (223.3, 40.0)
- added RA37001: 68kΩ, footprint:R0402, B.Cu at (184.9, 61.8)
- added RA38001: 68kΩ, footprint:R0402, B.Cu at (146.5, 40.0)
- added RA39001: 68kΩ, footprint:R0402, B.Cu at (108.0, 105.5)
- added RA40001: 68kΩ, footprint:R0402, B.Cu at (108.0, 83.7)
- added RA4001: 68kΩ, footprint:R0402, B.Cu at (165.7, 18.2)
- added RA41001: 68kΩ, footprint:R0402, B.Cu at (146.5, 83.7)
- added RA43001: 68kΩ, footprint:R0402, B.Cu at (165.7, 83.7)
- added RA44001: 68kΩ, footprint:R0402, B.Cu at (225.2, 126.7)
- added RA45001: 68kΩ, footprint:R0402, B.Cu at (204.1, 105.5)
- added RA46001: 68kΩ, footprint:R0402, B.Cu at (184.9, 83.7)
- added RA47001: 68kΩ, footprint:R0402, B.Cu at (127.3, 149.2)
- added RA48001: 68kΩ, footprint:R0402, B.Cu at (30.3, 115.7)
- added RA50001: 68kΩ, footprint:R0402, B.Cu at (165.7, 61.8)
- added RA5001: 68kΩ, footprint:R0402, B.Cu at (184.9, 105.5)
- added RA51001: 68kΩ, footprint:R0402, B.Cu at (53.3, 54.0)
- added RA52001: 68kΩ, footprint:R0402, B.Cu at (81.2, 58.9)
- added RA53001: 68kΩ, footprint:R0402, B.Cu at (108.0, 127.4)
- added RA56001: 68kΩ, footprint:R0402, B.Cu at (-52.5, 68.3)
- added RA57001: 68kΩ, footprint:R0402, B.Cu at (-33.3, 68.3)
- added RA58001: 68kΩ, footprint:R0402, B.Cu at (-33.3, 46.5)
- added RA59001: 68kΩ, footprint:R0402, B.Cu at (-52.5, 46.5)
- added RA6001: 68kΩ, footprint:R0402, B.Cu at (204.1, 18.2)
- added RA7001: 68kΩ, footprint:R0402, B.Cu at (165.7, 127.4)
- added RA8001: 68kΩ, footprint:R0402, B.Cu at (127.3, 83.7)
- added RA9001: 68kΩ, footprint:R0402, B.Cu at (146.5, 61.8)
- added RB10001: 33kΩ, footprint:R0402, B.Cu at (166.9, 149.2)
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Routing:
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Other:
- board outline removed

Commit message: Laying out the PCB.
Parts:
- removed C55003, C55004, C55005, C55006, C55008, C55011, CL12001, CL51001, CL57001, CL58001, CL59001, CL8001, CS12001, CS51001, CS57001, CS58001, CS59001, CS8001: 100nF, Capacitor_SMD:C_0402_1005Metric
- removed C55007: 10nF, Capacitor_SMD:C_0402_1005Metric
- removed C55009: 1uF, Capacitor_SMD:C_0402_1005Metric
- removed C55010: 4.7uF, Capacitor_SMD:C_0603_1608Metric
- removed J60002: Serial, Connector_PinHeader_2.54mm:PinHeader_1x05_P2.54mm_Vertical
- removed PB55002: TS-1187A-B-A-B, footprint:SW-SMD_4P-L5.1-W5.1-P3.70-LS6.5-TL-2
- removed R55005: 5.1k, Resistor_SMD:R_0402_1005Metric
- removed RA12001, RA51001, RA57001, RA58001, RA59001, RA8001: 68kΩ, footprint:R0402
- removed RB12001, RB51001, RB57001, RB58001, RB59001, RB8001: 33kΩ, footprint:R0402
- removed SR49001: 74HC165, Package_SO:SOIC-16_3.9x9.9mm_P1.27mm
- removed SW12001, SW51001, SW57001, SW58001, SW59001, SW8001: SW_Push, PCM_Switch_Keyboard_Hotswap_Kailh:SW_Hotswap_Kailh_MX
- removed U12001, U51001, U57001, U58001, U59001, U8001: SK6812MINI-E_C5149201, footprint:LED-SMD_L3.2-W2.8-TR
- added CL49001: 100nF, Capacitor_SMD:C_0402_1005Metric, B.Cu at (200.6, 132.3)
- added CS49001: 100nF, Capacitor_SMD:C_0402_1005Metric, B.Cu at (204.2, 132.5)
- added PB52001: TS-1187A-B-A-B, footprint:SW-SMD_4P-L5.1-W5.1-P3.70-LS6.5-TL-2, B.Cu at (31.8, 42.5)
- added RA49001: 68kΩ, footprint:R0402, B.Cu at (201.9, 133.0)
- added RB49001: 33kΩ, footprint:R0402, B.Cu at (202.9, 133.6)
- added SW49001: SW_Push, PCM_Switch_Keyboard_Hotswap_Kailh:SW_Hotswap_Kailh_MX, F.Cu at (196.8, 133.3)
- added U49001: SK6812MINI-E_C5149201, footprint:LED-SMD_L3.2-W2.8-TR, B.Cu at (199.4, 128.9)
- C55001, C55002, C55012, C55013, C55014, D55001, D55002, D55003, D55004, PB55001, R55001, R55002, R55003, R55004, R55007, R55008, R55009, R55010, SR15001, SR16001, SR29001, SR32001, SR42001, SR54001, STM55001, U55001, U55002, U55003, X55001: moved to B.Cu
- R55006: value 5.1k -> 7.7k; moved to B.Cu
- moved U60001 205.0 mm to (205.3, 61.6), turned to 90 degrees
- moved CS56001 198.2 mm to (134.1, 131.5), turned to 180 degrees
- moved RB56001 198.1 mm to (133.5, 133.1), turned to -90 degrees
- moved RA56001 195.8 mm to (132.3, 133.1), turned to 90 degrees
- moved D60001 194.8 mm to (197.5, 66.0)
- moved CL56001 193.2 mm to (130.9, 133.1), turned to 90 degrees
- moved J60003 192.4 mm to (177.8, 73.0), turned to 90 degrees
- moved U60002 190.2 mm to (195.6, 61.6)
- moved SW56001 189.9 mm to (128.1, 135.9), turned to 180 degrees
- moved U56001 186.4 mm to (128.1, 130.8), turned to 0 degrees
- moved CL10001 178.3 mm to (33.3, 28.3)
- moved CS10001 178.3 mm to (36.5, 26.7)
- moved RA10001 178.3 mm to (34.7, 28.3)
- moved RB10001 178.3 mm to (35.9, 28.3)
- moved SW10001 178.3 mm to (30.5, 31.1)
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Connections:
- CS23001 pad 2: /Left Half/5-Key Module/Key Unit12/SwitchOutput -> /Left Half/5-Key Module/Key Unit8/SwitchOutput
- CS41001 pad 2: /Left Half/5-Key Module/Key Unit11/SwitchOutput -> /Left Half/5-Key Module/Key Unit12/SwitchOutput
- CS43001 pad 2: /Left Half/5-Key Module/Key Unit10/SwitchOutput -> /Left Half/5-Key Module/Key Unit9/SwitchOutput
- CS56001 pad 2: /Left Half/5-Key Module1/Key Unit12/SwitchOutput -> /Left Half/5-Key Module/Key Unit10/SwitchOutput
- PB55001 pad 3: GND -> /Left Half/STM32 Module/BOOT0
- PB55001 pad 4: GND -> /Left Half/STM32 Module/BOOT0
- R55006 pad 1: Net-(R55005-Pad2) -> +5V
- RB23001 pad 1: /Left Half/5-Key Module/Key Unit12/SwitchOutput -> /Left Half/5-Key Module/Key Unit8/SwitchOutput
- RB41001 pad 1: /Left Half/5-Key Module/Key Unit11/SwitchOutput -> /Left Half/5-Key Module/Key Unit12/SwitchOutput
- RB43001 pad 1: /Left Half/5-Key Module/Key Unit10/SwitchOutput -> /Left Half/5-Key Module/Key Unit9/SwitchOutput
- RB56001 pad 1: /Left Half/5-Key Module1/Key Unit12/SwitchOutput -> /Left Half/5-Key Module/Key Unit10/SwitchOutput
- SR29001 pad 14: /Left Half/5-Key Module/Key Unit11/SwitchOutput -> /Left Half/5-Key Module/Key Unit12/SwitchOutput
- SR29001 pad 3: /Left Half/5-Key Module/Key Unit10/SwitchOutput -> /Left Half/5-Key Module/Key Unit13/SwitchOutput
- SR29001 pad 4: /Left Half/5-Key Module/Key Unit12/SwitchOutput -> /Left Half/5-Key Module/Key Unit9/SwitchOutput
- SR29001 pad 5: /Left Half/5-Key Module/Key Unit9/SwitchOutput -> /Left Half/5-Key Module/Key Unit8/SwitchOutput
- SR29001 pad 6: /Left Half/5-Key Module/Key Unit8/SwitchOutput -> /Left Half/5-Key Module/Key Unit10/SwitchOutput
- U23001 pad 2: /Left Half/5-Key Module/Key Unit10/LEDInput -> /Left Half/5-Key Module/Key Unit8/LEDOutput
- U23001 pad 4: /Left Half/5-Key Module/Key Unit12/LEDInput -> /Left Half/5-Key Module/Key Unit10/LEDOutput
- U41001 pad 4: /Left Half/5-Key Module/Key Unit10/LEDOutput -> /Left Half/5-Key Module/Key Unit12/LEDInput
- U43001 pad 2: /Left Half/5-Key Module/Key Unit10/LEDOutput -> /Left Half/5-Key Module/Key Unit13/LEDInput
- U43001 pad 4: /Left Half/5-Key Module/Key Unit10/LEDInput -> /Left Half/5-Key Module/Key Unit8/LEDOutput
- U56001 pad 2: /Left Half/5-Key Module1/Key Unit10/LEDInput -> /Left Half/5-Key Module/Key Unit10/LEDOutput
- U56001 pad 4: /Left Half/5-Key Module1/Key Unit12/LEDInput -> /Left Half/5-Key Module/LEDInput
Routing:
- net +3.3V: track 0.00 -> 78.4 mm, vias 0 -> 2
- net /Left Half/STM32 Module/BOOT0: track 0.00 -> 37.0 mm
- net /Left Half/STM32 Module/BOOT1: track 0.00 -> 25.8 mm
- net /Left Half/STM32 Module/ADC12_IN4: track 0.00 -> 14.6 mm, vias 0 -> 1
- net /Left Half/STM32 Module/NRST: track 0.00 -> 14.4 mm
- net +5V: track 675.3 -> 665.3 mm, vias 100 -> 92
- net /Left Half/STM32 Module/USBDP: track 0.00 -> 10.1 mm
- net Net-(STM55001-PD0): track 0.00 -> 8.98 mm
- net /Left Half/5-Key Module1/Key Unit10/LEDInput: track 8.26 -> 0.00 mm, vias 4 -> 0
- net /Left Half/5-Key Module/Key Unit10/LEDInput: track 8.26 -> 0.00 mm, vias 4 -> 0
- net /Left Half/5-Key Module1/Key Unit8/LEDOutput: track 8.26 -> 0.00 mm, vias 4 -> 0
- net /Left Half/5-Key Module1/Key Unit12/LEDInput: track 8.26 -> 0.00 mm, vias 4 -> 0
- net /Left Half/5-Key Module1/Key Unit10/LEDOutput: track 8.26 -> 0.00 mm, vias 4 -> 0
- net /Left Half/5-Key Module/Key Unit13/LEDInput: track 0.00 -> 8.26 mm, vias 0 -> 4
- net /Left Half/STM32 Module/USBDN: track 0.00 -> 7.89 mm
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Other:
- board outline added: 208.3 x 169.5 mm
